File: PCB/Faraway_PCB/Faraway_PCB.kicad_pcb (KiCad board)
At the start: 2 copper layers, 12 parts, among them J1 ESP32_DevKitV1_30PIN_Left, J2 ESP32_DevKitV1_30PIN_Right, Q1 PN2222A

Commit message: pcb ok
Parts:
- removed ISC2: Conn_01x02_Female, Connector_PinSocket_2.54mm:PinSocket_1x02_P2.54mm_Vertical
- removed RJ45_INPUT2: Conn_01x06_Female, Connector_PinHeader_2.54mm:PinHeader_1x06_P2.54mm_Vertical
- added I2C2: Conn_01x04_Female, Connector_PinSocket_2.54mm:PinSocket_1x04_P2.54mm_Vertical, F.Cu at (139.7, 86.4)
- I2C1: value Conn_01x02_Female -> Conn_01x04_Female; footprint Connector_PinSocket_2.54mm:PinSocket_1x02_P2.54mm_Vertical -> Connector_PinSocket_2.54mm:PinSocket_1x04_P2.54mm_Vertical
- moved RJ45_INPUT1 54.0 mm to (115.6, 101.6), turned to 90 degrees
- moved 5V_BONUS1 13.7 mm to (104.1, 48.3)
- moved R1 5.24 mm to (104.1, 91.4)
- moved HP1 5.08 mm to (104.1, 68.6)
- moved SK1 5.08 mm to (104.1, 58.4)
- moved Q1 3.81 mm to (104.1, 78.7)
- moved SPARE_PINS1 2.54 mm to (114.3, 76.2)
- moved J1 2.54 mm to (109.2, 55.9)
- moved J2 2.54 mm to (134.6, 55.9)
- moved I2C1 2.54 mm to (139.7, 71.1)
Connections:
- I2C1 pad 1: SCL -> +5V
- I2C1 pad 2: SDA -> SCL
- J1 pad 2: (no net) -> GND
- J2 pad 1: (no net) -> +5V
- Q1 pad 1: Net-(HP1-Pad2) -> GND
- Q1 pad 3: GND -> Net-(HP1-Pad2)
Routing:
- net PUL: track 0.00 -> 46.4 mm
- net DIR: track 0.00 -> 42.8 mm
- net EN: track 0.00 -> 39.2 mm
- net LED: track 0.00 -> 35.7 mm
- net SDA: track 0.00 -> 20.9 mm
- net SCL: track 0.00 -> 19.9 mm
- net SK: track 0.00 -> 10.4 mm
- net Net-(Q1-Pad2): track 0.00 -> 9.04 mm
- net AUDIO: track 0.00 -> 6.13 mm
- net Net-(J1-Pad9): track 0.00 -> 5.08 mm
- net Net-(J1-Pad11): track 0.00 -> 5.08 mm
- net Net-(J1-Pad10): track 0.00 -> 5.08 mm
- net Net-(HP1-Pad2): track 0.00 -> 5.08 mm
- added copper zone on B.Cu, net +5V
- added copper zone on F.Cu, net GND
Other:
- board outline added: 45.7 x 58.4 mm
- board text added: "D18"
- board text added: "D19"
- board text added: "D21"
- board text added: "Data"
- board text added: "ESP32 DEVKITV1 30Pin"
- board text added: "FAR AWAY"
- board text added: "HP+"
- board text added: "HP-"
- board text added: "Hémisphère / Chevalvert / 2021"
- board text added: "SCL"
- board text added: "SDA"
